File: shield.kicad_sch (KiCad schematic)
At the start: 8 parts, among them J1 DEVKIT_C2000_ROW_A, J2 DEVKIT_C2000_ROW_B, J3 NAPPE_ADC1, J4 NAPPE_ADC2, J5 NAPPE_PWM, J6 NAPPE_GPIO, J7 ALIM_5V, J8 ALIM_5V

Commit message: Versionne les librairies dans lib/ et la documentation dans doc/, imports/ reste la boite de reception
Parts:
- removed J1: DEVKIT_C2000_ROW_A, symbol c2000:DEVKIT_C2000_ROW_A
- removed J2: DEVKIT_C2000_ROW_B, symbol c2000:DEVKIT_C2000_ROW_B
- removed J3: NAPPE_ADC1, symbol c2000:NAPPE_ADC1
- removed J4: NAPPE_ADC2, symbol c2000:NAPPE_ADC2
- removed J5: NAPPE_PWM, symbol c2000:NAPPE_PWM
- removed J6: NAPPE_GPIO, symbol c2000:NAPPE_GPIO
- removed J7, J8: ALIM_5V, symbol c2000:ALIM_5V
- added J1: DEVKIT_C2000_ROW_A, symbol C2000_Devkit_Connectors:DEVKIT_C2000_ROW_A
- added J2: DEVKIT_C2000_ROW_B, symbol C2000_Devkit_Connectors:DEVKIT_C2000_ROW_B
- added J3: NAPPE_ADC1, symbol C2000_Devkit_Connectors:NAPPE_ADC1
- added J4: NAPPE_ADC2, symbol C2000_Devkit_Connectors:NAPPE_ADC2
- added J5: NAPPE_PWM, symbol C2000_Devkit_Connectors:NAPPE_PWM
- added J6: NAPPE_GPIO, symbol C2000_Devkit_Connectors:NAPPE_GPIO
- added J7, J8: ALIM_5V, symbol C2000_Devkit_Connectors:ALIM_5V
Connections:
- net +5V: now also J2.2 (+5V), J7.1 (+5V), J8.1 (+5V)
- net GND: now also J1.1 (GND), J1.13 (GND), J1.17 (GND), J1.20 (GND), J1.5 (GND), J1.9 (GND), J2.1 (GND), J2.14 (GND), J2.23 (GND), J2.9 (GND), J3.1 (GND), J3.11 (GND), J3.13 (GND), J3.15 (GND), J3.3 (GND), J3.5 (GND), J3.7 (GND), J3.9 (GND), J4.1 (GND), J4.11 (GND), J4.13 (GND), J4.15 (GND), J4.3 (GND), J4.5 (GND), J4.8 (GND), J4.9 (GND), J5.1 (GND), J5.11 (GND), J5.13 (GND), J5.15 (GND), J5.3 (GND), J5.5 (GND), J5.7 (GND), J5.9 (GND), J6.1 (GND), J6.11 (GND), J6.13 (GND), J6.15 (GND), J6.3 (GND), J6.5 (GND), J6.7 (GND), J6.9 (GND), J7.2 (GND), J8.2 (GND)

Commit message: Devkit en 2 x 28 et ESP32-C6-DevKitC-1 monte sur le shield (J9, J10)
Parts:
- added J10: ESP32_C6_DEVKITC_1_J3, symbol ESP32_C6_Devkit:ESP32_C6_DEVKITC_1_J3
- added J9: ESP32_C6_DEVKITC_1_J1, symbol ESP32_C6_Devkit:ESP32_C6_DEVKITC_1_J1
Connections:
- net +5V: now also J9.14 (+5V)
- net GND: now also J1.10 (GND), J1.16 (GND), J1.19 (GND), J1.21 (GND), J1.23 (GND), J1.25 (GND), J1.4 (GND), J1.7 (GND), J10.1 (GND), J10.12 (GND), J10.15 (GND), J9.15 (GND); no longer J1.17 (GND), J1.20 (GND), J1.5 (GND), J1.9 (GND)
Other:
- title: Shield d'isolation C2000 — connecteurs devkit et nappes -> Shield d'isolation C2000 — devkits, nappes et ESP32-C6
